File: irController.kicad_pcb (KiCad board)
At the start: 2 copper layers, 49 x 34 mm, 30 parts, among them P1 ZX62R-B-5P, P2 GPIO_USER, P3 WRITE_PROG, Q1 Q_NMOS, SW1 SKRPACE010, SW2 SKRPACE010, U1 NJM2845, U2 ESP-13-WROOM-02, U3 IRSNS_GP1UXC41QS

Commit message: 一旦完成
Parts:
- removed P3: WRITE_PROG, Socket_Strips:Socket_Strip_Straight_1x03
- added J1: B4B-PH-K-S(LF)(SN), SamacSys:SHDR4W60P0X200_1X4_990X450X600P, F.Cu at (169.5, 100.3)
- added R11: 22, Resistor_SMD:R_0603_1608Metric, F.Cu at (167.6, 94.5)
- added R12: 22, Resistor_SMD:R_0603_1608Metric, F.Cu at (165.6, 94.5)
- R1, R10, R2, R3, R4, R5, R6, R7, R8, R9: footprint Resistors_SMD:R_0603 -> Resistor_SMD:R_0603_1608Metric
- moved Q1 23.3 mm to (173.0, 72.0), turned to 0 degrees
- moved R5 15.4 mm to (151.9, 94.7), turned to 0 degrees
- moved R4 10.2 mm to (156.8, 91.9)
- moved C4 4.49 mm to (162.2, 94.6)
- moved R8 2.74 mm to (179.0, 78.7)
- moved D1 2.68 mm to (175.0, 78.7)
- moved D3 2.53 mm to (175.0, 93.5)
- moved R10 2.53 mm to (179.0, 93.5)
- moved R7 1.63 mm to (166.6, 83.3)
- moved R6 1.15 mm to (167.1, 78.0), turned to 180 degrees
- moved C3 0.71 mm to (141.5, 77.8)
- moved U2 0.08 mm to (146.1, 76.5)
Routing:
- net GND: track 234.9 -> 188.5 mm, vias 17 -> 11
- net Net-(C2-Pad1): track 96.4 -> 112.8 mm
- net Net-(Q1-Pad3): track 37.2 -> 25.5 mm
- net Net-(R11-Pad2): track 20.8 -> 11.4 mm, vias 1 -> 0
- net Net-(R12-Pad2): track 18.3 -> 9.16 mm, vias 1 -> 0
- net Net-(C4-Pad1): track 19.8 -> 13.4 mm, vias 2 -> 0
- net Net-(J1-Pad2): track 0.00 -> 5.12 mm
- net Net-(J1-Pad3): track 0.00 -> 5.06 mm
- net Net-(R6-Pad2): track 10.4 -> 7.88 mm
- net Net-(R4-Pad1): track 15.5 -> 14.2 mm
- net Net-(Q1-Pad1): track 18.4 -> 19.3 mm, vias 0 -> 2
Other:
- board text added: "GND/MISO/MOSI/VCC"
- board text removed: "GND/RX/TX"

Commit message: 発注時データ
Parts:
- added R13: 22, Resistor_SMD:R_0603_1608Metric, F.Cu at (147.0, 94.5)
- P1: footprint OriginalLibConn:USB_MICRO_HRS_ZX62R-B-5P -> Connector_USB:USB_Micro-B_Wuerth_629105150521
- moved R1 5.15 mm to (143.5, 94.5), turned to 0 degrees
- moved P1 3.78 mm to (143.5, 99.2)
- moved C2 2.67 mm to (144.2, 91.5), turned to 0 degrees
- renumbered SW1 to PROG
Connections:
- U2 pad 8: Net-(R1-Pad2) -> Net-(R13-Pad1)
Routing:
- net Net-(R13-Pad1): track 0.00 -> 17.2 mm
- net GND: track 188.5 -> 173.7 mm, vias 11 -> 14
- net Net-(R1-Pad2): track 21.5 -> 14.8 mm, vias 3 -> 2
- net Net-(C2-Pad1): track 112.8 -> 109.7 mm, vias 3 -> 1
- net Net-(C1-Pad1): track 15.7 -> 14.0 mm
Other:
- board text added: "(C) 2020 MolybYngFl"
- board text added: "IR Remote Controller V1.1"
- board text removed: "(C) 2017 MolybYngFl"
- board text removed: "IR Remote Controller V1.0"
